File: WiFi ROZETKA/untitled.brd (EAGLE design)
At the start: 55.9 x 61 mm, 25 parts, among them IC1 LM1117MP-3.3, IC2 LM1117MP-5.0, Q1 2N7002

Commit message: 26082017
Parts:
- JP1: value (none) -> ESP8266
- R1: value (none) -> 1k
- R2: value (none) -> 33k
- moved R2 18.8 mm to (54.6, 57.1), flipped to the bottom, turned to 180 degrees
- moved IC2 4.02 mm to (39.4, 48.3), flipped to the bottom
- moved Q1 2.84 mm to (54.6, 53.3), flipped to the bottom
- moved C2 2.54 mm to (47.0, 69.8), flipped to the bottom
- moved IC1 1.27 mm to (39.4, 68.6), flipped to the bottom
- flipped C1 to the bottom, turned to 0 degrees
- flipped D2 to the bottom, turned to 0 degrees
- turned PAD10 to 180 degrees
- turned PAD11 to 90 degrees
- turned PAD7 to 90 degrees
- flipped R1 to the bottom
Connections:
- removed net N$1: D2.C, PAD1.1, R2.2
- net +5V: now also D2.C, PAD1.1; no longer R2.1
- net GND: now also R2.2
- net N$3: now also R2.1
Routing:
- net N$17: track 70.1 -> 48.9 mm
- net +5V: track 100.5 -> 84.8 mm, vias 0 -> 1
- net +12V: track 16.7 -> 27.5 mm
- net N$16: track 8.89 -> 0.00 mm
- net N$1: track 7.09 -> 0.00 mm
- net N$4: track 75.8 -> 70.6 mm, vias 2 -> 0
- net GND: track 118.0 -> 119.4 mm
- net N$3: track 17.1 -> 18.2 mm, vias 4 -> 2
- net N$6: vias 0 -> 1
- net N$10: vias 0 -> 1
